Commit message: merged successfully, but still nee do adjust the parameters

File: grasp/hand.urdf (robot description, URDF)
Before this commit: robot hand3finger, 23 links, 22 joints
Joints:
- joint finger1-j1: origin xyz=0.016 0 0 rpy=0 0.3 0 -> xyz=0.016 0 0 rpy=0 0 0
- joint finger1-j2: origin xyz=0.054 0 0 rpy=0 0.3 0 -> xyz=0.054 0 0 rpy=0 0 0
- joint finger1-j3: origin xyz=0.0384 0 0 rpy=0 0.3 0 -> xyz=0.0384 0 0 rpy=0 0 0
- joint finger2-j1: origin xyz=0.016 0.0 0.0 rpy=0 0.3 0 -> xyz=0.016 0.0 0.0 rpy=0 0 0
- joint finger2-j2: origin xyz=0.054 0 0 rpy=0 0.3 0 -> xyz=0.054 0 0 rpy=0 0 0
- joint finger2-j3: origin xyz=0.0384 0 0 rpy=0 0.3 0 -> xyz=0.0384 0 0 rpy=0 0 0
- joint finger3-j1: origin xyz=0.016 0 0 rpy=0 0.3 0 -> xyz=0.016 0 0 rpy=0 0 0
- joint finger3-j2: origin xyz=0.054 0 0 rpy=0 0.3 0 -> xyz=0.054 0 0 rpy=0 0 0
- joint finger3-j3: origin xyz=0.0384 0 0 rpy=0 0.3 0 -> xyz=0.0384 0 0 rpy=0 0 0

Commit message: fix the bug of hand modeling

File: grasp/hand.urdf (robot description, URDF)
Before this commit: robot hand3finger, 23 links, 22 joints
Links:
- link finger0-link1: geometry visual box size=0.016 0.018 0.025
Joints:
- joint finger0-j0: origin xyz=-0.0155 -0.015 -0.008 rpy=0.1 0 0 -> xyz=-0.0155 0.015 -0.008 rpy=0 0 -0.087
- joint finger0-j1: origin xyz=-0.01 -0.036 0 rpy=0 0.1 0 -> xyz=-0.01 0.036 0 rpy=0 -0.25 0
- joint finger0-j2: origin xyz=0 -0.015 0 rpy=0 0 0.2 -> xyz=0 0.018 0 rpy=0 0 1.57
- joint finger0-j3: origin xyz=0.05 0 0 rpy=0 0 0.2 -> xyz=0.05 0 0 rpy=0 0 0
- joint finger1-j1: origin xyz=0.016 0 0 rpy=0 0 0 -> xyz=0.016 0 0 rpy=0 0.3 0
- joint finger1-j2: origin xyz=0.054 0 0 rpy=0 0 0 -> xyz=0.054 0 0 rpy=0 0.3 0
- joint finger1-j3: origin xyz=0.0384 0 0 rpy=0 0 0 -> xyz=0.0384 0 0 rpy=0 0.3 0
- joint finger2-j1: origin xyz=0.016 0.0 0.0 rpy=0 0 0 -> xyz=0.016 0.0 0.0 rpy=0 0.3 0
- joint finger2-j2: origin xyz=0.054 0 0 rpy=0 0 0 -> xyz=0.054 0 0 rpy=0 0.3 0
- joint finger2-j3: origin xyz=0.0384 0 0 rpy=0 0 0 -> xyz=0.0384 0 0 rpy=0 0.3 0
- joint finger3-j1: origin xyz=0.016 0 0 rpy=0 0 0 -> xyz=0.016 0 0 rpy=0 0.3 0
- joint finger3-j2: origin xyz=0.054 0 0 rpy=0 0 0 -> xyz=0.054 0 0 rpy=0 0.3 0
- joint finger3-j3: origin xyz=0.0384 0 0 rpy=0 0 0 -> xyz=0.0384 0 0 rpy=0 0.3 0

Commit message: update the bug in the hand model: the number index and the 3-finger orientation

File: grasp/hand.urdf (robot description, URDF)
Before this commit: robot hand3finger, 23 links, 22 joints
Joints:
- joint finger1-j0: origin xyz=0.0475 -0.041 -0.015 rpy=0 0 0 -> xyz=0.0475 0.041 -0.015 rpy=0 0 0.0872
- joint finger3-j0: origin xyz=0.0475 0.041 -0.015 rpy=0 0 0 -> xyz=0.0475 -0.041 -0.015 rpy=0 0 -0.0872

Commit message: the version before we update the thumb model

File: grasp/hand.urdf (robot description, URDF)
Before this commit: robot hand3finger, 23 links, 22 joints
Joints:
- joint finger0-j0: origin xyz=-0.0155 0.015 -0.008 rpy=0 0 -0.087 -> xyz=-0.0155 0.015 -0.008 rpy=0 0 0.087

Commit message: fix the bug in normal detection, and this is the version before we modify on the thumb

File: grasp/hand.urdf (robot description, URDF)
Before this commit: robot hand3finger, 23 links, 22 joints
Joints:
- joint finger1-j1: origin xyz=0.016 0 0 rpy=0 0.3 0 -> xyz=0.016 0 0 rpy=0 0.0 0
- joint finger1-j2: origin xyz=0.054 0 0 rpy=0 0.3 0 -> xyz=0.054 0 0 rpy=0 0.0 0
- joint finger1-j3: origin xyz=0.0384 0 0 rpy=0 0.3 0 -> xyz=0.0384 0 0 rpy=0 0.0 0
- joint finger2-j1: origin xyz=0.016 0.0 0.0 rpy=0 0.3 0 -> xyz=0.016 0.0 0.0 rpy=0 0.0 0
- joint finger2-j2: origin xyz=0.054 0 0 rpy=0 0.3 0 -> xyz=0.054 0 0 rpy=0 0.0 0
- joint finger2-j3: origin xyz=0.0384 0 0 rpy=0 0.3 0 -> xyz=0.0384 0 0 rpy=0 0.0 0
- joint finger3-j1: origin xyz=0.016 0 0 rpy=0 0.3 0 -> xyz=0.016 0 0 rpy=0 0.0 0
- joint finger3-j2: origin xyz=0.054 0 0 rpy=0 0.3 0 -> xyz=0.054 0 0 rpy=0 0.0 0
- joint finger3-j3: origin xyz=0.0384 0 0 rpy=0 0.3 0 -> xyz=0.0384 0 0 rpy=0 0.0 0

Commit message: modified the thumb finger model

File: grasp/hand.urdf (robot description, URDF)
Before this commit: robot hand3finger, 23 links, 22 joints
Joints:
- joint finger0-j0: origin xyz=-0.0155 0.015 -0.008 rpy=0 0 0.087 -> xyz=0.002513 0.01933 0.0032 rpy=0 0 0.087
- joint finger0-j1: origin xyz=-0.01 0.036 0 rpy=0 -0.25 0 -> xyz=-0.028 0.038 -0.0034 rpy=0 -0.25 0
- joint finger0-j2: origin xyz=0 0.018 0 rpy=0 0 1.57 -> xyz=0 0.0175 0 rpy=0 0 1.57
- joint finger0-j3: origin xyz=0.05 0 0 rpy=0 0 0 -> xyz=0.052 0 0 rpy=0 0 0

Commit message: add i controller to the position pid control

File: grasp/hand.urdf (robot description, URDF)
Before this commit: robot hand3finger, 23 links, 22 joints
Links:
- link finger0-link0: geometry visual box size=0.036 0.045 0.036
Joints:
- joint finger0-j1: origin xyz=-0.028 0.038 -0.0034 rpy=0 -0.25 0 -> xyz=-0.028 0.038 -0.0034 rpy=0 0.25 0

Commit message: the version can be reversed to before discriminating thumb normal detection

File: grasp/hand.urdf (robot description, URDF)
Before this commit: robot hand3finger, 23 links, 22 joints
Joints:
- joint finger1-j0: origin xyz=0.0475 0.041 -0.015 rpy=0 0 0.0872 -> xyz=0.0455 0.041 -0.015 rpy=0 0 0.0872
- joint finger3-j0: origin xyz=0.0475 -0.041 -0.015 rpy=0 0 -0.0872 -> xyz=0.0455 -0.041 -0.015 rpy=0 0 -0.0872

Commit message: update velocity saturation and bounce back in the applying force back. but the surface normal is still predefined just for debugging

File: grasp/hand.urdf (robot description, URDF)
Before this commit: robot hand3finger, 23 links, 22 joints
Links:
- link finger0-link0: mass 0.0716 -> 0.1
- link finger0-link1: mass 0.01 -> 0.001
- link finger0-link2: mass 0.0509 -> 0.03
- link finger0-link3: mass 0.047 -> 0.05
- link finger1-link0: mass 0.0716 -> 0.001
- link finger1-link1: mass 0.0716 -> 0.3
- link finger1-link2: mass 0.0509 -> 0.04
- link finger1-link3: mass 0.047 -> 0.09
- link finger2-link0: mass 0.0716 -> 0.001
- link finger2-link1: mass 0.0716 -> 0.3
- link finger2-link2: mass 0.0509 -> 0.04
- link finger2-link3: mass 0.047 -> 0.09
- link finger3-link0: mass 0.0716 -> 0.001
- link finger3-link1: mass 0.0716 -> 0.3
- link finger3-link2: mass 0.0509 -> 0.04
- link finger3-link3: mass 0.047 -> 0.09

Commit message: a huge progress, debug the error in the joint angle offset, and implement the joint control for the pregrasp

File: grasp/hand.urdf (robot description, URDF)
Before this commit: robot hand3finger, 23 links, 22 joints
Joints:
- joint finger0-j1: origin xyz=-0.028 0.038 -0.0034 rpy=0 0.25 0 -> xyz=-0.028 0.038 -0.0034 rpy=0 0 0
